File: 3.7-5/3.7LiPoly Management.sch (EAGLE design)
At the start: 32 parts, among them J1 DX4R005HJ5R2000, J2 S2B-PH-SM4-TB(LF)(SN), T1 MMUN2133LT1G, U1 TPS61090RSAR, U2 MCP73871T-2CCI/ML

Commit message: Update
Getting more familiar with Git and updating cleanly
Parts:
- renumbered U$1 to L1, U$3 to H1
Changed lines of the file:
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@@
 <part name="R4" library="rcl" library_urn="urn:adsk.eagle:library:334" deviceset="R-US_" device="R0805" package3d_urn="urn:adsk.eagle:package:23553/2" value="1.87M"/>
 <part name="R5" library="rcl" library_urn="urn:adsk.eagle:library:334" deviceset="R-US_" device="R0805" package3d_urn="urn:adsk.eagle:package:23553/2" value="200K"/>
-<part name="U$1" library="VLCF5020T-6R8N1R1" deviceset="VLCF5020T" device="" value="6.8uH"/>
+<part name="L1" library="VLCF5020T-6R8N1R1" deviceset="VLCF5020T" device="" value="6.8uH"/>
 <part name="C4" library="rcl" library_urn="urn:adsk.eagle:library:334" deviceset="C-US" device="C0805" package3d_urn="urn:adsk.eagle:package:23617/2" value="2.2uF"/>
 <part name="C5" library="rcl" library_urn="urn:adsk.eagle:library:334" deviceset="C-US" device="C0805" package3d_urn="urn:adsk.eagle:package:23617/2" value="100uF"/>
@@
 <part name="U$2" library="JS102011SAQN" deviceset="JS102011SAQN" device=""/>
 <part name="GND18" library="supply1" library_urn="urn:adsk.eagle:library:371" deviceset="GND" device=""/>
-<part name="U$3" library="M22-6340442" deviceset="M22-6340442" device=""/>
+<part name="H1" library="M22-6340442" deviceset="M22-6340442" device=""/>
 <part name="GND19" library="supply1" library_urn="urn:adsk.eagle:library:371" deviceset="GND" device=""/>
 <part name="CHARGE" library="KingBright" deviceset="WP934AD" device="" value="YELLOW"/>
@@
 <attribute name="VALUE" x="153.162" y="34.29" size="1.778" layer="96" rot="R90"/>
 </instance>
-<instance part="U$1" gate="A" x="27.94" y="53.34" smashed="yes">
+<instance part="L1" gate="A" x="27.94" y="53.34" smashed="yes">
 <attribute name="VALUE" x="25.9588" y="49.0728" size="3.4798" layer="96" ratio="10" rot="SR0"/>
 <attribute name="NAME" x="27.0256" y="56.6928" size="3.4798" layer="95" ratio="10" rot="SR0"/>
@@
 <attribute name="VALUE" x="101.6" y="10.16" size="1.778" layer="96"/>
 </instance>
-<instance part="U$3" gate="A" x="271.78" y="55.88" smashed="yes"/>
+<instance part="H1" gate="A" x="271.78" y="55.88" smashed="yes"/>
 <instance part="GND19" gate="1" x="271.78" y="35.56" smashed="yes">
 <attribute name="VALUE" x="269.24" y="33.02" size="1.778" layer="96"/>
@@
 <segment>
 <pinref part="GND19" gate="1" pin="GND"/>
-<pinref part="U$3" gate="A" pin="P2"/>
+<pinref part="H1" gate="A" pin="P2"/>
 <wire x1="271.78" y1="38.1" x2="271.78" y2="45.72" width="0.1524" layer="91"/>
 </segment>
@@
 <wire x1="261.62" y1="43.18" x2="261.62" y2="50.8" width="0.1524" layer="91"/>
 <label x="261.62" y="50.8" size="1.778" layer="95" rot="R90" xref="yes"/>
-<pinref part="U$3" gate="A" pin="P1"/>
+<pinref part="H1" gate="A" pin="P1"/>
 <wire x1="269.24" y1="45.72" x2="269.24" y2="43.18" width="0.1524" layer="91"/>
 <wire x1="269.24" y1="43.18" x2="261.62" y2="43.18" width="0.1524" layer="91"/>
@@
 </segment>
 <segment>
-<pinref part="U$1" gate="A" pin="2"/>
+<pinref part="L1" gate="A" pin="2"/>
 <wire x1="27.94" y1="53.34" x2="22.86" y2="53.34" width="0.1524" layer="91"/>
 <label x="22.86" y="53.34" size="1.778" layer="95" rot="R180" xref="yes"/>
@@
 <wire x1="48.26" y1="71.12" x2="48.26" y2="53.34" width="0.1524" layer="91"/>
 <junction x="48.26" y="53.34"/>
-<pinref part="U$1" gate="A" pin="1"/>
+<pinref part="L1" gate="A" pin="1"/>
 <wire x1="48.26" y1="53.34" x2="43.18" y2="53.34" width="0.1524" layer="91"/>
 </segment>
