File: RPi Zero W Breakout/RPi Zero W Breakout 0.3.sch (EAGLE design)
At the start: 35 parts, among them J1 35RAPC4BHN2

Commit message: Update
minor layer changes for text
Parts:
- renumbered PIN1 to J2, U$3 to H1
Changed lines of the file:
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@@
 </classes>
 <parts>
-<part name="PIN1" library="con-hirose" library_urn="urn:adsk.eagle:library:152" deviceset="FH12-10S-0.5S" device="H" package3d_urn="urn:adsk.eagle:package:7323/1"/>
+<part name="J2" library="con-hirose" library_urn="urn:adsk.eagle:library:152" deviceset="FH12-10S-0.5S" device="H" package3d_urn="urn:adsk.eagle:package:7323/1"/>
 <part name="J1" library="35RAPC4BHN2" deviceset="35RAPC4BHN2" device=""/>
 <part name="C2" library="rcl" library_urn="urn:adsk.eagle:library:334" deviceset="C-US" device="C0805K" package3d_urn="urn:adsk.eagle:package:23681/2" value="33n"/>
@@
 <part name="GND1" library="supply1" library_urn="urn:adsk.eagle:library:371" deviceset="GND" device=""/>
 <part name="GND2" library="supply1" library_urn="urn:adsk.eagle:library:371" deviceset="GND" device=""/>
-<part name="U$3" library="M22-6340442" deviceset="M22-6340442" device=""/>
+<part name="H1" library="M22-6340442" deviceset="M22-6340442" device=""/>
 <part name="U$2" library="LM4810MM" deviceset="LM4810MM/NOPBCT-ND" device=""/>
 <part name="RSPK" library="SP-1208" deviceset="SP-1208" device=""/>
@@
 </plain>
 <instances>
-<instance part="PIN1" gate="-1" x="205.74" y="73.66" smashed="yes">
+<instance part="J2" gate="-1" x="205.74" y="73.66" smashed="yes">
 <attribute name="NAME" x="207.772" y="72.898" size="1.778" layer="95"/>
 <attribute name="VALUE" x="195.58" y="76.2" size="1.778" layer="96"/>
 </instance>
-<instance part="PIN1" gate="-2" x="205.74" y="71.12" smashed="yes">
+<instance part="J2" gate="-2" x="205.74" y="71.12" smashed="yes">
 <attribute name="NAME" x="207.772" y="70.358" size="1.778" layer="95"/>
 </instance>
-<instance part="PIN1" gate="-3" x="205.74" y="68.58" smashed="yes">
+<instance part="J2" gate="-3" x="205.74" y="68.58" smashed="yes">
 <attribute name="NAME" x="207.772" y="67.818" size="1.778" layer="95"/>
 </instance>
-<instance part="PIN1" gate="-4" x="205.74" y="66.04" smashed="yes">
+<instance part="J2" gate="-4" x="205.74" y="66.04" smashed="yes">
 <attribute name="NAME" x="207.772" y="65.278" size="1.778" layer="95"/>
 </instance>
-<instance part="PIN1" gate="-5" x="205.74" y="63.5" smashed="yes">
+<instance part="J2" gate="-5" x="205.74" y="63.5" smashed="yes">
 <attribute name="NAME" x="207.772" y="62.738" size="1.778" layer="95"/>
 </instance>
-<instance part="PIN1" gate="-6" x="205.74" y="60.96" smashed="yes">
+<instance part="J2" gate="-6" x="205.74" y="60.96" smashed="yes">
 <attribute name="NAME" x="207.772" y="60.198" size="1.778" layer="95"/>
 </instance>
-<instance part="PIN1" gate="-7" x="205.74" y="58.42" smashed="yes">
+<instance part="J2" gate="-7" x="205.74" y="58.42" smashed="yes">
 <attribute name="NAME" x="207.772" y="57.658" size="1.778" layer="95"/>
 </instance>
-<instance part="PIN1" gate="-8" x="205.74" y="55.88" smashed="yes">
+<instance part="J2" gate="-8" x="205.74" y="55.88" smashed="yes">
 <attribute name="NAME" x="207.772" y="55.118" size="1.778" layer="95"/>
 </instance>
-<instance part="PIN1" gate="-9" x="205.74" y="53.34" smashed="yes">
+<instance part="J2" gate="-9" x="205.74" y="53.34" smashed="yes">
 <attribute name="NAME" x="207.772" y="52.578" size="1.778" layer="95"/>
 </instance>
-<instance part="PIN1" gate="-10" x="205.74" y="50.8" smashed="yes">
+<instance part="J2" gate="-10" x="205.74" y="50.8" smashed="yes">
 <attribute name="NAME" x="207.772" y="50.038" size="1.778" layer="95"/>
 </instance>
@@
 <attribute name="VALUE" x="73.66" y="142.24" size="1.778" layer="96"/>
 </instance>
-<instance part="U$3" gate="A" x="43.18" y="73.66" smashed="yes" rot="R270"/>
+<instance part="H1" gate="A" x="43.18" y="73.66" smashed="yes" rot="R270"/>
 <instance part="U$2" gate="G$1" x="119.38" y="147.32" smashed="yes" rot="R90"/>
 <instance part="RSPK" gate="G$1" x="215.9" y="132.08" smashed="yes"/>
@@
 <net name="LEDK" class="0">
 <segment>
-<pinref part="PIN1" gate="-1" pin="1"/>
+<pinref part="J2" gate="-1" pin="1"/>
 <wire x1="198.12" y1="73.66" x2="203.2" y2="73.66" width="0.1524" layer="91"/>
 <label x="198.12" y="73.66" size="1.27" layer="95" rot="R180" xref="yes"/>
@@
 <net name="MISO" class="0">
 <segment>
-<pinref part="PIN1" gate="-2" pin="1"/>
+<pinref part="J2" gate="-2" pin="1"/>
 <wire x1="198.12" y1="71.12" x2="203.2" y2="71.12" width="0.1524" layer="91"/>
 <label x="198.12" y="71.12" size="1.27" layer="95" rot="R180" xref="yes"/>
@@
 <net name="CS" class="0">
 <segment>
-<pinref part="PIN1" gate="-5" pin="1"/>
+<pinref part="J2" gate="-5" pin="1"/>
 <wire x1="203.2" y1="63.5" x2="198.12" y2="63.5" width="0.1524" layer="91"/>
 <label x="198.12" y="63.5" size="1.27" layer="95" rot="R180" xref="yes"/>
@@
 <net name="RESET" class="0">
 <segment>
-<pinref part="PIN1" gate="-8" pin="1"/>
+<pinref part="J2" gate="-8" pin="1"/>
 <wire x1="203.2" y1="55.88" x2="198.12" y2="55.88" width="0.1524" layer="91"/>
 <label x="198.12" y="55.88" size="1.27" layer="95" rot="R180" xref="yes"/>
@@
 </segment>
 <segment>
-<pinref part="PIN1" gate="-9" pin="1"/>
+<pinref part="J2" gate="-9" pin="1"/>
 <wire x1="203.2" y1="53.34" x2="198.12" y2="53.34" width="0.1524" layer="91"/>
 <label x="198.12" y="53.34" size="1.27" layer="95" rot="R180" xref="yes"/>
@@
 </segment>
 <segment>
-<pinref part="U$3" gate="A" pin="P4"/>
+<pinref part="H1" gate="A" pin="P4"/>
 <wire x1="33.02" y1="68.58" x2="27.94" y2="68.58" width="0.1524" layer="91"/>
 </segment>
@@
 <net name="GND" class="0">
 <segment>
-<pinref part="PIN1" gate="-10" pin="1"/>
+<pinref part="J2" gate="-10" pin="1"/>
 <wire x1="203.2" y1="50.8" x2="198.12" y2="50.8" width="0.1524" layer="91"/>
 <label x="198.12" y="50.8" size="1.27" layer="95" rot="R180" xref="yes"/>
@@
 </segment>
 <segment>
-<pinref part="U$3" gate="A" pin="P3"/>
+<pinref part="H1" gate="A" pin="P3"/>
 <wire x1="33.02" y1="71.12" x2="27.94" y2="71.12" width="0.1524" layer="91"/>
 </segment>
@@
 </segment>
 <segment>
-<pinref part="PIN1" gate="-4" pin="1"/>
+<pinref part="J2" gate="-4" pin="1"/>
 <wire x1="203.2" y1="66.04" x2="198.12" y2="66.04" width="0.1524" layer="91"/>
 <label x="198.12" y="66.04" size="1.27" layer="95" rot="R180" xref="yes"/>
@@
 </segment>
 <segment>
-<pinref part="PIN1" gate="-3" pin="1"/>
+<pinref part="J2" gate="-3" pin="1"/>
 <wire x1="203.2" y1="68.58" x2="198.12" y2="68.58" width="0.1524" layer="91"/>
 <label x="198.12" y="68.58" size="1.27" layer="95" rot="R180" xref="yes"/>
@@
 </segment>
 <segment>
-<pinref part="PIN1" gate="-7" pin="1"/>
+<pinref part="J2" gate="-7" pin="1"/>
 <wire x1="203.2" y1="58.42" x2="198.12" y2="58.42" width="0.1524" layer="91"/>
 <label x="198.12" y="58.42" size="1.27" layer="95" rot="R180" xref="yes"/>
